File: esp-testhw.sch (KiCad schematic (older format))
At the start: 21 parts

Commit message: Finished schematic draft
Parts:
- removed L? (x2): RF FERRITE, symbol INDUCTOR
- removed P?: CONN_01X03, symbol CONN_01X03
- removed R?: 220R, FT:RES_CAY16, symbol R_PACK4
- removed R?: 10K, symbol R
- added C3: 22uF X5R 16V, FT:1210_CAP, symbol CAP
- added C5: 100nF 6.3V, FT:0603_CAP, symbol CAP
- added L1, L2, L3: BLM18KG121TN1D, FT:0603, symbol INDUCTOR
- added P3: CONN_01X02, FT:1X02, symbol CONN_01X02
- added R4: 220R, FT:RES_CAY16, symbol R_PACK4
- added R5: 10K, FT:RES_CAY16, symbol R_PACK4
- added SW1, SW2: SW_PUSHBUTTON, FT:SW_PUSHBUTTON_SMD, symbol SW_PUSHBUTTON
- C1, C2, C6, C7: renamed from C?; value 22uF 10V -> 22uF X5R 16V
- gave numbers to parts that had none: 12
Connections:
- net labels added: A_GPIO13_UART_RX, A_GPIO15_UART_TX, A_VCC, B_GPIO15_UART_TX, B_VCC, PWM_OUT, STM_VCC, STM_~RST
- net labels removed: A_UART_RX, A_UART_TX, BOOT_PULL, B_AIN, B_UART_TX, SWD_~RST
- wire segments 124 -> 155
- no-connect marks 14 -> 17
Other:
- note added: "ESP8266 A"
- note added: "ESP8266 B"
- note added: "ESP8266\nSoftware i2c"
- note added: "HSPI CLK"
- note added: "HSPI MISO"
- note added: "HSPI MOSI\n"
- note added: "HSPI ~CS"
- note added: "I2SI_BCK\n"
- note added: "I2SI_DATA"
- note added: "I2SI_WS"
- note added: "I2SO_DATA"
- note added: "Pulling A_GPIO0 for bootloader\nalso pulls B_GPIO0"
- note added: "STM Bootloader Button"
- note added: "STM Bootloader Jumper\n"
- note added: "STM Reset Button"
- note removed: "STM Boot Mode Select"
- note removed: "Test Device A"
- note removed: "Test Device B"
- moved on the sheet: P2, R3, U2
